File: Pcb2/CA6/_autosave-CA6_2.kicad_pcb (KiCad board)
At the start: 2 copper layers, 101.6 x 170.2 mm, 130 parts, among them J1 MICRO_USB, J2 BAT_CON, J3 MODULE_0, J4 MODULE_2, J5 MODULE_1, J6 AUX, J7 AUX, J8 MODULE_3, P1 JTAG, P2 RFD22301 Breakout, Q1 BSS138P, Q10 BSS138P, Q11 BSS138P, Q12 BSS138P, Q13 BSS138P, Q14 BSS138P, Q15 BSS138P, Q16 BSS138P, Q2 BSS138P, Q3 BSS138P, Q4 BSS138P, Q5 BSS138P, Q6 BSS138P, Q7 BSS138P, Q8 BSS138P, Q9 BSS138P, SW1 ERASE, SW2 USB/BATTERY, SW3 RESET, U1 L_PIPE, U12 VREG_33, U14 EEPROM, U15 L_PIPE, U16 ATSAM3X8EA-AU_LQFP-144, U2 L_PIPE, U3 L_PIPE, U4 L_PIPE, U5 L_PIPE, U6 L_PIPE, U7 L_PIPE, U8 L_PIPE, X1 HOLE, X2 HOLE, X3 HOLE, X4 HOLE, X7 CRYSTAL_4, X8 32khz

Commit message: More updates on pcb layout
Other:
- copper layers 2 -> 4
- board text removed: "Inner1 Copper - Layer 2"
- board text removed: "Inner2 Copper - Layer 3"
Changed lines of the file:
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@@
   (general
     (links 398)
-    (no_connects 0)
+    (no_connects 7)
     (area 22.672669 23.322669 129.727331 195.9824)
     (thickness 1.6)
-    (drawings 19)
+    (drawings 17)
     (tracks 2430)
     (zones 0)
@@
   (layers
     (0 F.Cu signal)
+    (1 In1.Cu signal)
+    (2 In2.Cu signal)
     (31 B.Cu signal)
     (34 B.Paste user)
@@
       (net 23 /AUX24))
   )
-  (module CA6:SLP3-150-100-R (layer F.Cu)
-    (at 124.46 153.67 90)
-    (fp_text reference U15 (at -3.556 2.159 90) (layer F.SilkS)
-      (effects (font (size 0.8 0.8) (thickness 0.15)))
-    )
-    (fp_text value L_PIPE (at 0 -2.032 90) (layer F.SilkS) hide
-      (effects (font (size 0.2286 0.381) (thickness 0.0508)))
-    )
-    (fp_line (start -2.0426 1.6984) (end -2.2606 1.6984) (layer F.SilkS) (width 0.14986))
-    (fp_line (start 1.5 3.54) (end 1.5 2.5) (layer F.SilkS) (width 0.14986))
-    (fp_line (start -1.5 3.54) (end -1.5 2.5) (layer F.SilkS) (width 0.14986))
-    (fp_arc (start 0 3.54) (end 1.5 3.54) (angle 180) (layer F.SilkS) (width 0.14986))
-    (fp_line (start 2.25 2.5) (end 2.25 1.8) (layer F.SilkS) (width 0.14986))
-    (fp_line (start -2.25 1.8) (end -2.25 2.5) (layer F.SilkS) (width 0.14986))
-    (fp_line (start -2.25 2.5) (end 2.25 2.5) (layer F.SilkS) (width 0.14986))
-    (fp_line (start -2.25 1.8) (end -2.25 -1.8) (layer F.SilkS) (width 0.14986))
-    (fp_line (start -2.25 -1.8) (end 2.25 -1.8) (layer F.SilkS) (width 0.14986))
-    (fp_line (start 2.25 -1.8) (end 2.25 1.8) (layer F.SilkS) (width 0.14986))
-    (fp_line (start 2.25 1.8) (end 2.032 1.8) (layer F.SilkS) (width 0.14986))
-    (pad "" np_thru_hole circle (at 1.25 -2.7 90) (size 1.1684 1.1684) (drill 1.1684) (layers *.Cu *.Mask F.SilkS))
-    (pad "" np_thru_hole circle (at -1.25 -2.7 90) (size 1.1684 1.1684) (drill 1.1684) (layers *.Cu *.Mask F.SilkS))
-  )
   (module CA6:SOT-23_11AA160 (layer F.Cu)
     (at 63.5 121.412 270)
@@
       (net 96 /VDDOUT))
   )
+  (module CA6:SLP3-150-100-R (layer F.Cu)
+    (at 124.46 153.67 90)
+    (fp_text reference U15 (at -3.556 2.159 90) (layer F.SilkS)
+      (effects (font (size 0.8 0.8) (thickness 0.15)))
+    )
+    (fp_text value L_PIPE (at 0 -2.032 90) (layer F.SilkS) hide
+      (effects (font (size 0.2286 0.381) (thickness 0.0508)))
+    )
+    (fp_line (start -2.0426 1.6984) (end -2.2606 1.6984) (layer F.SilkS) (width 0.14986))
+    (fp_line (start 1.5 3.54) (end 1.5 2.5) (layer F.SilkS) (width 0.14986))
+    (fp_line (start -1.5 3.54) (end -1.5 2.5) (layer F.SilkS) (width 0.14986))
+    (fp_arc (start 0 3.54) (end 1.5 3.54) (angle 180) (layer F.SilkS) (width 0.14986))
+    (fp_line (start 2.25 2.5) (end 2.25 1.8) (layer F.SilkS) (width 0.14986))
+    (fp_line (start -2.25 1.8) (end -2.25 2.5) (layer F.SilkS) (width 0.14986))
+    (fp_line (start -2.25 2.5) (end 2.25 2.5) (layer F.SilkS) (width 0.14986))
+    (fp_line (start -2.25 1.8) (end -2.25 -1.8) (layer F.SilkS) (width 0.14986))
+    (fp_line (start -2.25 -1.8) (end 2.25 -1.8) (layer F.SilkS) (width 0.14986))
+    (fp_line (start 2.25 -1.8) (end 2.25 1.8) (layer F.SilkS) (width 0.14986))
+    (fp_line (start 2.25 1.8) (end 2.032 1.8) (layer F.SilkS) (width 0.14986))
+    (pad "" np_thru_hole circle (at 1.25 -2.7 90) (size 1.1684 1.1684) (drill 1.1684) (layers *.Cu *.Mask F.SilkS))
+    (pad "" np_thru_hole circle (at -1.25 -2.7 90) (size 1.1684 1.1684) (drill 1.1684) (layers *.Cu *.Mask F.SilkS))
+  )
   (gr_line (start 114.3 167.64) (end 111.76 167.64) (angle 90) (layer F.SilkS) (width 0.2032))
   (gr_line (start 114.3 195.58) (end 114.3 167.64) (angle 90) (layer F.SilkS) (width 0.2032))
@@
     (effects (font (size 0.95758 0.95758) (thickness 0.2032)) (justify left))
   )
-  (gr_text "Inner2 Copper - Layer 3" (at 31.75 168.91) (layer In2.Cu)
-    (effects (font (size 1.50114 1.50114) (thickness 0.29972)) (justify left))
-  )
-  (gr_text "Inner1 Copper - Layer 2" (at 31.75 166.37) (layer In1.Cu)
-    (effects (font (size 1.50114 1.50114) (thickness 0.29972)) (justify left))
-  )
   (gr_line (start 121.92 25.4) (end 30.48 25.4) (angle 90) (layer Edge.Cuts) (width 0.09906))
   (gr_line (start 127 190.5) (end 127 30.48) (angle 90) (layer Edge.Cuts) (width 0.09906))
@@
       )
     )
-  )
-  (zone (net 0) (net_name "") (layer In2.Cu) (hatch edge 0.508)
-    (connect_pads (clearance 0.508))
-    (min_thickness 0.254)
-    (keepout (tracks not_allowed) (vias not_allowed) (copperpour allowed))
-    (fill (arc_segments 16) (thermal_gap 0.508) (thermal_bridge_width 0.508))
-    (polygon
-      (pts
-        (xy 43.942 48.006) (xy 25.4 48.006) (xy 25.4 47.498) (xy 43.942 47.498)
-      )
-    )
-  )
-  (zone (net 100) (net_name GND) (layer In1.Cu) (hatch edge 0.508)
-    (connect_pads (clearance 0.254))
-    (min_thickness 0.254)
-    (fill yes (mode segment) (arc_segments 32) (thermal_gap 0.508) (thermal_bridge_width 0.508))
-    (polygon
-      (pts
-        (xy 106.426 135.128) (xy 104.394 135.128) (xy 104.4067 141.2367) (xy 87.122 141.224) (xy 87.122 153.1874)
-        (xy 88.0237 154.9527) (xy 88.0364 159.639) (xy 88.0237 159.639) (xy 85.5218 159.639) (xy 45.72 159.639)
-        (xy 45.6565 32.004) (xy 106.3625 32.004)
-      )
-    )
