File: Pcb2/CA6/CA6.kicad_pcb (KiCad board)
At the start: 2 copper layers, 101.6 x 170.2 mm, 130 parts, among them J1 MICRO_USB, J2 BAT_CON, J3 MODULE_0, J4 MODULE_2, J5 MODULE_1, J6 AUX, J7 AUX, J8 MODULE_3, P1 JTAG, P2 RFD22301 Breakout, Q1 BSS138P, Q10 BSS138P, Q11 BSS138P, Q12 BSS138P, Q13 BSS138P, Q14 BSS138P, Q15 BSS138P, Q16 BSS138P, Q2 BSS138P, Q3 BSS138P, Q4 BSS138P, Q5 BSS138P, Q6 BSS138P, Q7 BSS138P, Q8 BSS138P, Q9 BSS138P, SW1 ERASE, SW2 USB/BATTERY, SW3 RESET, U1 L_PIPE, U12 VREG_33, U14 EEPROM, U15 L_PIPE, U16 ATSAM3X8EA-AU_LQFP-144, U2 L_PIPE, U3 L_PIPE, U4 L_PIPE, U5 L_PIPE, U6 L_PIPE, U7 L_PIPE, U8 L_PIPE, X1 HOLE, X2 HOLE, X3 HOLE, X4 HOLE, X7 CRYSTAL_4, X8 32khz

Commit message: Routing pcb
Parts:
- moved C30 9.61 mm to (110.5, 50.2)
- moved C3 7.91 mm to (55.9, 141.5)
- moved C38 7.75 mm to (55.9, 139.6)
- moved C31 7.62 mm to (110.5, 119.4)
- moved C32 5.72 mm to (110.5, 74.3)
- moved C37 3.17 mm to (110.5, 98.4)
Connections:
- J6 pad 1: /AUX00 -> /AUX_TX
- J6 pad 2: /AUX01 -> /AUX_RX
- J6 pad 45: /AUX_TX -> /AUX44
- J6 pad 46: /AUX_RX -> /AUX45
- J6 pad 47: GND -> /AUX46
- J6 pad 48: 3V3 -> /AUX47
- J7 pad 1: /AUX00 -> /AUX_TX
- J7 pad 2: /AUX01 -> /AUX_RX
- J7 pad 45: /AUX_TX -> /AUX44
- J7 pad 46: /AUX_RX -> /AUX45
- J7 pad 47: GND -> /AUX46
- J7 pad 48: 3V3 -> /AUX47
- P2 pad 10: (no net) -> /CC_PROG
- P2 pad 8: (no net) -> /CC_RESET
- U16 pad 1: /CAM2S -> /CAM1S
- U16 pad 100: /AUX25 -> /AUX29
- U16 pad 101: /AUX24 -> /AUX28
- U16 pad 102: /AUX23 -> /AUX27
- U16 pad 103: /AUX22 -> /AUX26
- U16 pad 112: /AUX21 -> /AUX25
- U16 pad 113: /AUX20 -> /AUX24
- U16 pad 114: /AUX19 -> /AUX23
- U16 pad 115: /AUX18 -> /AUX22
- U16 pad 116: /AUX17 -> /AUX21
- U16 pad 117: /AUX16 -> /AUX20
- U16 pad 118: /AUX15 -> /AUX19
- U16 pad 119: /AUX14 -> /AUX18
- U16 pad 120: /AUX13 -> /AUX17
- U16 pad 121: /AUX12 -> /AUX16
- U16 pad 122: /AUX11 -> /AUX15
- U16 pad 123: /AUX10 -> /AUX14
- U16 pad 127: /AUX09 -> /AUX13
- U16 pad 128: /AUX08 -> /AUX12
- U16 pad 13: (no net) -> /CAM2F
- U16 pad 131: /AUX07 -> /AUX11
- U16 pad 132: /AUX06 -> /AUX10
- U16 pad 133: /AUX05 -> /AUX09
- U16 pad 134: /AUX04 -> /AUX08
- U16 pad 135: /AUX03 -> /AUX07
- U16 pad 136: /AUX02 -> /AUX06
- U16 pad 137: /AUX01 -> /AUX05
- U16 pad 138: /AUX00 -> /AUX04
- U16 pad 14: (no net) -> /CAM2S
- U16 pad 140: /CAM0F -> /AUX03
- U16 pad 141: /CAM0S -> /AUX02
- U16 pad 142: /CAM1F -> /CAM0F
- U16 pad 143: /CAM1S -> /CAM0S
- U16 pad 144: /CAM2F -> /CAM1F
- U16 pad 55: /MOD3_ID -> /CC_RESET
- U16 pad 59: (no net) -> /CC_PROG
- U16 pad 60: (no net) -> /MOD3_ID
- U16 pad 66: /AUX43 -> /AUX47
- U16 pad 67: /AUX42 -> /AUX46
- U16 pad 68: /AUX41 -> /AUX45
- U16 pad 71: /AUX40 -> /AUX44
- U16 pad 72: /AUX39 -> /AUX43
- U16 pad 76: /AUX38 -> /AUX42
- U16 pad 77: /AUX37 -> /AUX41
- U16 pad 89: /AUX36 -> /AUX40
- U16 pad 90: /AUX35 -> /AUX39
- U16 pad 91: /AUX34 -> /AUX38
- U16 pad 92: /AUX33 -> /AUX37
- U16 pad 93: /AUX32 -> /AUX36
- U16 pad 94: /AUX31 -> /AUX35
- U16 pad 95: /AUX30 -> /AUX34
- U16 pad 96: /AUX29 -> /AUX33
- U16 pad 97: /AUX28 -> /AUX32
- U16 pad 98: /AUX27 -> /AUX31
- U16 pad 99: /AUX26 -> /AUX30
Routing:
- net 3V3: track 11.6 -> 403.7 mm, vias 2 -> 9
- net /UOTGID: track 0.00 -> 65.8 mm, vias 0 -> 2
- net /VBUS: track 18.6 -> 74.1 mm, vias 0 -> 4
- net Net-(C42-Pad1): track 0.00 -> 8.46 mm
- net GND: track 163.9 -> 171.9 mm, vias 72 -> 79
- net Net-(C15-Pad1): track 0.00 -> 7.92 mm
- net (no net): track 0.00 -> 1.91 mm
- net /D+: track 44.5 -> 43.3 mm
- added copper zone on F.Cu, net GND
Other:
- board text removed: "Back Copper - Layer 2"
- board text removed: "Back Silk Screen - Layer 5"
- board text removed: "Back Solder Mask - Layer 7"
- board text removed: "Back Solder Paste - Layer 3"
- board text removed: "Board Edge Cut - Layer 12"
- board text removed: "Front Copper - Layer 1"
- board text removed: "Front Silk Screen - Layer 6"
- board text removed: "Front Solder Mask - Layer 8"
- board text removed: "Front Solder Paste - Layer 4"

Commit message: More updates on pcb layout
Parts:
- P2: footprint Socket_Strips:Socket_Strip_Straight_2x05_Pitch2.54mm -> Socket_Strips:Socket_Strip_Straight_1x10_Pitch2.54mm
- moved C23 26.5 mm to (119.4, 157.5)
- moved P2 21.9 mm to (121.9, 160.0), turned to 0 degrees
- moved C34 21.6 mm to (116.3, 156.5)
- moved R22 9.91 mm to (124.3, 148.8)
- moved R30 9.91 mm to (121.8, 148.8)
- moved D1 8.89 mm to (124.5, 144.8)
- moved U15 8.89 mm to (124.5, 144.8)
- moved C19 0.74 mm to (85.2, 137.3)
- moved C21 0.68 mm to (85.2, 142.7)
- moved C40 0.65 mm to (85.2, 138.8)
Routing:
- net GND: track 171.9 -> 165.2 mm, vias 79 -> 75
- net 3V3: track 403.7 -> 408.8 mm, vias 9 -> 10
- net (no net): track 1.91 -> 0.00 mm
- net /VBUS: track 74.1 -> 75.4 mm
- net /UOTGID: vias 2 -> 4
Other:
- board text added: "Connection Card"
- board text removed: "Inner1 Copper - Layer 2"
- board text removed: "Inner2 Copper - Layer 3"

Commit message: Another layout of the pcb
Connections:
- P2 pad 10: /CC_PROG -> /CC_RX
- P2 pad 3: /CC_RX -> /CC_R_LED
- P2 pad 4: Net-(P2-Pad4) -> /CC_G_LED
- P2 pad 5: /CC_TX -> /CC_PROG
- P2 pad 6: Net-(P2-Pad6) -> /CC_RESET
- P2 pad 7: /CC_RTS -> /CC_CTS
- P2 pad 8: /CC_RESET -> /CC_RTS
- P2 pad 9: /CC_CTS -> /CC_TX
- R22 pad 1: Net-(P2-Pad6) -> /CC_G_LED
- R30 pad 1: Net-(P2-Pad4) -> /CC_R_LED
Routing:
- net /UOTGID: track 65.8 -> 4.47 mm, vias 4 -> 0
- net GND: track 165.2 -> 197.6 mm, vias 75 -> 70
- net Net-(C14-Pad1): track 18.1 -> 3.13 mm
- net Net-(C17-Pad1): track 11.5 -> 5.77 mm
- net /VDDOUT: track 0.00 -> 3.03 mm
- net Net-(C20-Pad1): track 0.00 -> 1.50 mm
- net /VBUS: track 75.4 -> 75.9 mm
