File: Pcb2/CA6/CA6.kicad_pcb (KiCad board)
At the start: 2 copper layers, 101.6 x 170.2 mm, 130 parts, among them J1 MICRO_USB, J2 BAT_CON, J3 MODULE_0, J4 MODULE_2, J5 MODULE_1, J6 AUX, J7 AUX, J8 MODULE_3, P1 JTAG, P2 RFD22301 Breakout, Q1 BSS138P, Q10 BSS138P, Q11 BSS138P, Q12 BSS138P, Q13 BSS138P, Q14 BSS138P, Q15 BSS138P, Q16 BSS138P, Q2 BSS138P, Q3 BSS138P, Q4 BSS138P, Q5 BSS138P, Q6 BSS138P, Q7 BSS138P, Q8 BSS138P, Q9 BSS138P, SW1 ERASE, SW2 USB/BATTERY, SW3 RESET, U1 L_PIPE, U12 VREG_33, U14 EEPROM, U15 L_PIPE, U16 ATSAM3X8EA-AU_LQFP-144, U2 L_PIPE, U3 L_PIPE, U4 L_PIPE, U5 L_PIPE, U6 L_PIPE, U7 L_PIPE, U8 L_PIPE, X1 HOLE, X2 HOLE, X3 HOLE, X4 HOLE, X7 CRYSTAL_4, X8 32khz

Commit message: Check in pcb files
Parts:
- removed J7: AUX, CA6:IDC_50PIN(2X25)-M
- P2: value RFD22301 Breakout -> Connection Card
- SW2: value USB/BATTERY -> USB / BATTERY
- moved SW1 12.7 mm to (51.4, 109.2), turned to 180 degrees
- moved SW3 12.7 mm to (101.0, 109.2), turned to 180 degrees
- moved BT1 11.4 mm to (76.2, 73.7)
- moved C23 9.40 mm to (119.1, 148.1)
- moved C34 9.40 mm to (116.3, 147.1)
- moved R29 8.13 mm to (72.6, 114.0)
- moved C1 7.62 mm to (86.2, 133.1)
- moved C10 7.62 mm to (63.2, 116.4)
- moved C11 7.62 mm to (66.0, 148.6)
- moved C12 7.62 mm to (72.6, 118.6)
- moved C14 7.62 mm to (72.1, 154.7)
- moved C15 7.62 mm to (78.2, 119.4)
- moved C17 7.62 mm to (76.0, 154.7)
- moved C19 7.62 mm to (85.2, 129.7)
- moved C20 7.62 mm to (82.2, 147.7)
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Routing:
- net GND: track 197.6 -> 202.4 mm, vias 70 -> 74
- net 3V3: track 408.8 -> 404.0 mm
Other:
- board size 101.6 x 170.2 mm -> 101.6 x 162.6 mm
- board text added: "+ -"
- board text added: "3.3V"
- board text added: "CTS"
- board text added: "Camera Axe 6 Version 4 March 9, 2017"
- board text added: "G_LED"
- board text added: "Gnd"
- board text added: "PROG"
- board text added: "RESET"
- board text added: "RTS"
- board text added: "RX"
- board text added: "R_LED"
- board text added: "TX"
- board text removed: "Camera Axe 6 Version 4 March 3, 2017"

Commit message: Clean up file names for pcb
Routing:
- net /CC_RTS: track 0.00 -> 172.0 mm, vias 0 -> 1
- net /MOD1_SCL: track 0.00 -> 157.4 mm
- net /AUX_RX: track 0.00 -> 148.1 mm, vias 0 -> 2
- net /MOD0_ID: track 0.00 -> 134.3 mm
- net /AUX04: track 0.00 -> 129.2 mm
- net /MOD0_RX: track 0.00 -> 128.6 mm, vias 0 -> 3
- net /CAM1S: track 0.00 -> 127.0 mm
- net /CAM2S: track 0.00 -> 124.8 mm, vias 0 -> 2
- net /MOD0_TX: track 0.00 -> 123.6 mm, vias 0 -> 4
- net /MOD0_SCL: track 0.00 -> 122.4 mm, vias 0 -> 1
- net /AUX_TX: track 0.00 -> 122.0 mm
- net /MOD1_TX: track 0.00 -> 119.0 mm, vias 0 -> 2
- net /AUX11: track 0.00 -> 118.8 mm
- net /MOD1_RX: track 0.00 -> 117.9 mm, vias 0 -> 2
- net /CAM0S: track 0.00 -> 117.4 mm, vias 0 -> 2
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