File: Pcb2/CA6/CA6.sch (KiCad schematic (older format))
At the start: 130 parts, among them J1 MICRO_USB, J2 BAT_CON, J3 MODULE_0, J4 MODULE_2, J5 MODULE_1, J6 AUX, J7 AUX, J8 MODULE_3, P1 JTAG, P2 RFD22301 Breakout, Q1 BSS138P, Q10 BSS138P, Q11 BSS138P, Q12 BSS138P, Q13 BSS138P, Q14 BSS138P, Q15 BSS138P, Q16 BSS138P, Q2 BSS138P, Q3 BSS138P, Q4 BSS138P, Q5 BSS138P, Q6 BSS138P, Q7 BSS138P, Q8 BSS138P, Q9 BSS138P, SW1 ERASE, SW2 USB/BATTERY, SW3 RESET, U1 L_PIPE, U12 VREG_33, U14 EEPROM, U15 L_PIPE, U16 ATSAM3X8EA-AU_LQFP-144, U2 L_PIPE, U3 L_PIPE, U4 L_PIPE, U5 L_PIPE, U6 L_PIPE, U7 L_PIPE, U8 L_PIPE, X1 HOLE, X2 HOLE, X3 HOLE, X4 HOLE, X7 CRYSTAL_4, X8 32khz

Commit message: Another layout of the pcb
Connections:
- net CC_CTS: now also P2.7 (PIN7); no longer P2.9 (PIN9)
- net CC_PROG: now also P2.5 (PIN5); no longer P2.10 (PIN10)
- net CC_RESET: now also P2.6 (PIN6); no longer P2.8 (PIN8)
- net CC_RTS: now also P2.8 (PIN8); no longer P2.7 (PIN7)
- net CC_RX: now also P2.10 (PIN10); no longer P2.3 (PIN3)
- net CC_TX: now also P2.9 (PIN9); no longer P2.5 (PIN5)
- net CC_G_LED: now reaches R22.1
- net CC_G_LED: now also P2.4 (PIN4); no longer P2.6 (PIN6)
- net CC_R_LED: now reaches R30.1
- net CC_R_LED: now also P2.3 (PIN3); no longer P2.4 (PIN4)
Other:
- moved on the sheet: D1, R22, R30, U15
Changed lines of the file:
@@
 L R R22
 U 1 1 535CC0F4
-P 20550 13250
-F 0 "R22" V 20630 13250 40  0000 C CNN
-F 1 "680R" V 20557 13251 40  0000 C CNN
-F 2 "CA6:SM0603_Resistor" V 20480 13250 30  0001 C CNN
-F 3 "~" H 20550 13250 30  0000 C CNN
-	1    20550 13250
+P 21100 13150
+F 0 "R22" V 21180 13150 40  0000 C CNN
+F 1 "680R" V 21107 13151 40  0000 C CNN
+F 2 "CA6:SM0603_Resistor" V 21030 13150 30  0001 C CNN
+F 3 "~" H 21100 13150 30  0000 C CNN
+	1    21100 13150
 	0    -1   -1   0
 $EndComp
@@
 L LED_LIGHT_PIPE U15
 U 1 1 5372AFB0
-P 21600 13150
-F 0 "U15" H 21600 13350 60  0000 C CNN
-F 1 "L_PIPE" H 21600 12940 60  0000 C CNN
-F 2 "CA6:SLP3-150-100-R" H 21600 13150 60  0001 C CNN
-F 3 "~" H 21600 13150 60  0000 C CNN
-	1    21600 13150
+P 22150 13050
+F 0 "U15" H 22150 13250 60  0000 C CNN
+F 1 "L_PIPE" H 22150 12840 60  0000 C CNN
+F 2 "CA6:SLP3-150-100-R" H 22150 13050 60  0001 C CNN
+F 3 "~" H 22150 13050 60  0000 C CNN
+	1    22150 13050
 	1    0    0    -1
 $EndComp
@@
 L R R30
 U 1 1 5424B8EF
-P 20550 12950
-F 0 "R30" V 20630 12950 40  0000 C CNN
-F 1 "680R" V 20557 12951 40  0000 C CNN
-F 2 "CA6:SM0603_Resistor" V 20480 12950 30  0001 C CNN
-F 3 "~" H 20550 12950 30  0000 C CNN
-	1    20550 12950
+P 21100 12850
+F 0 "R30" V 21180 12850 40  0000 C CNN
+F 1 "680R" V 21107 12851 40  0000 C CNN
+F 2 "CA6:SM0603_Resistor" V 21030 12850 30  0001 C CNN
+F 3 "~" H 21100 12850 30  0000 C CNN
+	1    21100 12850
 	0    -1   -1   0
 $EndComp
@@
 L LED2C D1
 U 1 1 542537D2
-P 21150 13100
-F 0 "D1" H 21105 13410 50  0000 C CNN
-F 1 "LED2C" H 21300 13000 50  0000 C CNN
-F 2 "CA6:LED-SOT-23" V 20985 13270 60  0001 C CNN
-F 3 "~" V 20985 13270 60  0000 C CNN
-	1    21150 13100
+P 21700 13000
+F 0 "D1" H 21655 13310 50  0000 C CNN
+F 1 "LED2C" H 21850 12900 50  0000 C CNN
+F 2 "CA6:LED-SOT-23" V 21535 13170 60  0001 C CNN
+F 3 "~" V 21535 13170 60  0000 C CNN
+	1    21700 13000
 	0    -1   -1   0
 $EndComp
@@
 Wire Wire Line
 	18200 13250 17750 13250
-Text Label 17850 12950 0    60   ~ 0
-CC_RX
-Text Label 17850 13050 0    60   ~ 0
+Text Label 17750 13250 0    60   ~ 0
 CC_TX
-Text Label 17850 13150 0    60   ~ 0
+Text Label 20150 13150 2    60   ~ 0
 CC_RTS
-Text Label 17850 13250 0    60   ~ 0
+Text Label 17750 13150 0    60   ~ 0
 CC_CTS
 Wire Wire Line
@@
 Wire Wire Line
 	19700 13250 20150 13250
-Text Label 19750 13150 0    60   ~ 0
+Text Label 19750 13050 0    60   ~ 0
 CC_RESET
-Text Label 19750 13250 0    60   ~ 0
+Text Label 17750 13050 0    60   ~ 0
 CC_PROG
 $Comp
 L GND #PWR093
 U 1 1 58CBFA9E
-P 21300 13100
-F 0 "#PWR093" H 21300 13100 30  0001 C CNN
-F 1 "GND" H 21300 13030 30  0001 C CNN
-F 2 "" H 21300 13100 60  0000 C CNN
-F 3 "" H 21300 13100 60  0000 C CNN
-	1    21300 13100
-	1    0    0    -1
-$EndComp
-Connection ~ 21300 13100
-Connection ~ 20800 12950
-Connection ~ 20800 13250
-Wire Wire Line
-	19700 12950 20300 12950
-Wire Wire Line
-	19700 13050 20300 13050
-Wire Wire Line
-	20300 13050 20300 13250
-Connection ~ 20300 13250
-Connection ~ 20300 12950
+P 21850 13000
+F 0 "#PWR093" H 21850 13000 30  0001 C CNN
+F 1 "GND" H 21850 12930 30  0001 C CNN
+F 2 "" H 21850 13000 60  0000 C CNN
+F 3 "" H 21850 13000 60  0000 C CNN
+	1    21850 13000
+	1    0    0    -1
+$EndComp
+Connection ~ 21850 13000
+Connection ~ 21350 12850
+Connection ~ 21350 13150
 Wire Wire Line
 	19700 12850 20200 12850
@@
 Text Label 16450 3200 0    60   ~ 0
 AUX47
+Wire Wire Line
+	20850 12850 20500 12850
+Wire Wire Line
+	20850 13150 20500 13150
+Text Label 20500 12850 0    60   ~ 0
+CC_R_LED
+Text Label 20500 13150 0    60   ~ 0
+CC_G_LED
+Wire Wire Line
+	19700 12950 20150 12950
+Wire Wire Line
+	19700 13050 20150 13050
+Text Label 20150 13250 2    60   ~ 0
+CC_RX
+Text Label 17750 12950 0    60   ~ 0
+CC_R_LED
+Text Label 19750 12950 0    60   ~ 0
+CC_G_LED
 $EndSCHEMATC

Commit message: Check in pcb files
Parts:
- removed J7: AUX, CA6:IDC_50PIN(2X25)-M, symbol IDC_50PIN(2X25)
- P2: value RFD22301 Breakout -> Connection Card
Other:
- note added: "Connection Card"
- note removed: "Connectivity Card"
- moved on the sheet: C33, J6
