File: Pcb2/CA6/CA6_2.kicad_pcb (KiCad board)
At the start: 2 copper layers, 101.6 x 170.2 mm, 130 parts, among them J1 MICRO_USB, J2 BAT_CON, J3 MODULE_0, J4 MODULE_2, J5 MODULE_1, J6 AUX, J7 AUX, J8 MODULE_3, P1 JTAG, P2 RFD22301 Breakout, Q1 BSS138P, Q10 BSS138P, Q11 BSS138P, Q12 BSS138P, Q13 BSS138P, Q14 BSS138P, Q15 BSS138P, Q16 BSS138P, Q2 BSS138P, Q3 BSS138P, Q4 BSS138P, Q5 BSS138P, Q6 BSS138P, Q7 BSS138P, Q8 BSS138P, Q9 BSS138P, SW1 ERASE, SW2 USB/BATTERY, SW3 RESET, U1 L_PIPE, U12 VREG_33, U14 EEPROM, U15 L_PIPE, U16 ATSAM3X8EA-AU_LQFP-144, U2 L_PIPE, U3 L_PIPE, U4 L_PIPE, U5 L_PIPE, U6 L_PIPE, U7 L_PIPE, U8 L_PIPE, X1 HOLE, X2 HOLE, X3 HOLE, X4 HOLE, X7 CRYSTAL_4, X8 32khz

Commit message: More updates on pcb layout
Parts:
- P2: footprint Socket_Strips:Socket_Strip_Straight_2x05_Pitch2.54mm -> Socket_Strips:Socket_Strip_Straight_1x10_Pitch2.54mm
- moved C23 26.5 mm to (119.4, 157.5)
- moved P2 21.9 mm to (121.9, 160.0), turned to 0 degrees
- moved C34 21.6 mm to (116.3, 156.5)
- moved R22 9.91 mm to (124.3, 148.8)
- moved R30 9.91 mm to (121.8, 148.8)
- moved D1 8.89 mm to (124.5, 144.8)
- moved U15 8.89 mm to (124.5, 144.8)
- moved C19 0.74 mm to (85.2, 137.3)
- moved C21 0.68 mm to (85.2, 142.7)
- moved C40 0.65 mm to (85.2, 138.8)
Routing:
- net /MOD0_TX: track 250.5 -> 0.00 mm
- net /AUX_RX: track 158.9 -> 0.00 mm, vias 10 -> 0
- net /CC_CTS: track 149.2 -> 0.00 mm, vias 13 -> 0
- net /MOD0_ID: track 147.8 -> 0.00 mm
- net /AUX_TX: track 126.4 -> 0.00 mm, vias 6 -> 0
- net /AUX11: track 124.0 -> 0.00 mm
- net /AUX03: track 122.0 -> 0.00 mm
- net /MOD1_TX: track 120.1 -> 0.00 mm, vias 2 -> 0
- net /AUX02: track 119.9 -> 0.00 mm
- net /AUX05: track 119.8 -> 0.00 mm
- net /MOD1_RX: track 119.7 -> 0.00 mm, vias 2 -> 0
- net /MOD0_RX: track 119.4 -> 0.00 mm, vias 3 -> 0
- net /AUX09: track 119.3 -> 0.00 mm
- net /AUX07: track 118.9 -> 0.00 mm, vias 1 -> 0
- net /AUX15: track 118.5 -> 0.00 mm, vias 3 -> 0
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Other:
- board text added: "Connection Card"
- board text removed: "Inner1 Copper - Layer 2"
- board text removed: "Inner2 Copper - Layer 3"

Commit message: Another layout of the pcb
Connections:
- P2 pad 10: /CC_PROG -> /CC_RX
- P2 pad 3: /CC_RX -> /CC_R_LED
- P2 pad 4: Net-(P2-Pad4) -> /CC_G_LED
- P2 pad 5: /CC_TX -> /CC_PROG
- P2 pad 6: Net-(P2-Pad6) -> /CC_RESET
- P2 pad 7: /CC_RTS -> /CC_CTS
- P2 pad 8: /CC_RESET -> /CC_RTS
- P2 pad 9: /CC_CTS -> /CC_TX
- R22 pad 1: Net-(P2-Pad6) -> /CC_G_LED
- R30 pad 1: Net-(P2-Pad4) -> /CC_R_LED
Routing:
- net /CAM3S: track 0.00 -> 176.3 mm
- net /CAM3F: track 0.00 -> 174.5 mm
- net /AUX_TX: track 0.00 -> 152.7 mm
- net /MOD0_RX: track 0.00 -> 152.3 mm, vias 0 -> 2
- net /MOD0_TX: track 0.00 -> 149.5 mm, vias 0 -> 2
- net /CC_RTS: track 0.00 -> 147.9 mm, vias 0 -> 1
- net /AUX_RX: track 0.00 -> 140.7 mm, vias 0 -> 2
- net /M_RESET: track 0.00 -> 127.1 mm, vias 0 -> 3
- net /MOD0_SCL: track 0.00 -> 126.6 mm, vias 0 -> 1
- net /AUX21: track 0.00 -> 125.7 mm, vias 0 -> 2
- net /AUX14: track 0.00 -> 124.3 mm, vias 0 -> 3
- net /AUX03: track 0.00 -> 122.0 mm
- net /AUX02: track 0.00 -> 119.9 mm
- net /AUX05: track 0.00 -> 119.8 mm
- net /MOD0_SDA: track 0.00 -> 119.8 mm, vias 0 -> 1
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
Commit message: Check in pcb files
Parts:
- removed J7: AUX, CA6:IDC_50PIN(2X25)-M
- P2: value RFD22301 Breakout -> Connection Card
- SW2: value USB/BATTERY -> USB / BATTERY
- moved SW1 12.7 mm to (51.4, 109.2), turned to 180 degrees
- moved SW3 12.7 mm to (101.0, 109.2), turned to 180 degrees
- moved BT1 11.4 mm to (76.2, 73.7)
- moved C23 9.40 mm to (119.1, 148.1)
- moved C34 9.40 mm to (116.3, 147.1)
- moved R29 8.13 mm to (72.6, 114.0)
- moved C1 7.62 mm to (86.2, 133.1)
- moved C10 7.62 mm to (63.2, 116.4)
- moved C11 7.62 mm to (66.0, 148.6)
- moved C12 7.62 mm to (72.6, 118.6)
- moved C13 7.62 mm to (77.3, 116.8)
- moved C14 7.62 mm to (72.1, 154.7)
- moved C15 7.62 mm to (78.2, 119.4)
- moved C17 7.62 mm to (76.0, 154.7)
- moved C19 7.62 mm to (85.2, 129.7)
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Routing:
- net /CAM3S: track 176.3 -> 80.4 mm, vias 0 -> 4
- net /MOD1_SCL: track 82.2 -> 157.4 mm, vias 1 -> 0
- net /CAM3F: track 174.5 -> 103.2 mm, vias 0 -> 2
- net /MOD0_ID: track 99.2 -> 134.3 mm, vias 1 -> 0
- net /M_RESET: track 127.1 -> 94.8 mm, vias 3 -> 5
- net /AUX_TX: track 152.7 -> 122.0 mm
- net /CAM7F: track 48.6 -> 78.8 mm, vias 2 -> 0
- net /CAM2S: track 96.1 -> 124.8 mm
- net /MOD0_TX: track 149.5 -> 123.6 mm, vias 2 -> 4
- net /CC_RTS: track 147.9 -> 172.0 mm
- net /MOD0_RX: track 152.3 -> 128.6 mm, vias 2 -> 3
- net /AUX21: track 125.7 -> 102.1 mm
- net /MOD2_AN4: track 60.9 -> 83.9 mm, vias 3 -> 2
- net /AUX14: track 124.3 -> 101.7 mm, vias 3 -> 2
- net 3V3: track 442.0 -> 420.8 mm, vias 12 -> 10
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Other:
- board size 101.6 x 170.2 mm -> 101.6 x 162.6 mm
- board text added: "+ -"
- board text added: "3.3V"
- board text added: "CTS"
- board text added: "Camera Axe 6 Version 4 March 9, 2017"
- board text added: "G_LED"
- board text added: "Gnd"
- board text added: "PROG"
- board text added: "RESET"
- board text added: "RTS"
- board text added: "RX"
- board text added: "R_LED"
- board text added: "TX"
- board text removed: "Camera Axe 6 Version 4 March 3, 2017"
