File: Pcb/CA6_0.kicad_pcb (KiCad board)
At the start: 2 copper layers, 101.6 x 162.6 mm, 129 parts, among them J1 MICRO_USB, J2 BAT_CON, J3 MODULE_0, J4 MODULE_2, J5 MODULE_1, J6 AUX, J8 MODULE_3, P1 JTAG, P2 Connection Card, Q1 BSS138P, Q10 BSS138P, Q11 BSS138P, Q12 BSS138P, Q13 BSS138P, Q14 BSS138P, Q15 BSS138P, Q16 BSS138P, Q2 BSS138P, Q3 BSS138P, Q4 BSS138P, Q5 BSS138P, Q6 BSS138P, Q7 BSS138P, Q8 BSS138P, Q9 BSS138P, SW1 ERASE, SW2 USB / BATTERY, SW3 RESET, U1 L_PIPE, U12 VREG_33, U14 EEPROM, U15 L_PIPE, U16 ATSAM3X8EA-AU_LQFP-144, U2 L_PIPE, U3 L_PIPE, U4 L_PIPE, U5 L_PIPE, U6 L_PIPE, U7 L_PIPE, U8 L_PIPE, X1 HOLE, X2 HOLE, X3 HOLE, X4 HOLE, X7 CRYSTAL_4, X8 32khz

Commit message: Update gerbers and remove logo off back of pcb
Parts:
- removed LOGO2: CA_LOGO_150, CA6:CA_Logo_15mm
- SW2: value USB / BATTERY -> USB/BATTERY
Other:
- board text added: "Camera Axe 6 Version 4 March 10, 2017"
- board text removed: "Camera Axe 6 Version 4 March 9, 2017"

Commit message: Update card header to have 2 more pins -- now a 6x2 header
Parts:
- added X5: HOLE, CA6:HOLE_3.0mm, F.Cu at (86.4, 156.2)
- P2: value Connection Card -> Connection_Card; footprint Socket_Strips:Socket_Strip_Straight_1x10_Pitch2.54mm -> Socket_Strips:Socket_Strip_Straight_2x06_Pitch2.54mm
- moved P2 3.82 mm to (122.2, 156.2)
- moved Q2 1.27 mm to (40.6, 68.6), turned to 90 degrees
Connections:
- U16 pad 1: /CAM1S -> /CAM1F
- U16 pad 100: /AUX29 -> /AUX31
- U16 pad 101: /AUX28 -> /AUX30
- U16 pad 102: /AUX27 -> /AUX29
- U16 pad 103: /AUX26 -> /AUX28
- U16 pad 112: /AUX25 -> /AUX27
- U16 pad 113: /AUX24 -> /AUX26
- U16 pad 114: /AUX23 -> /AUX25
- U16 pad 115: /AUX22 -> /AUX24
- U16 pad 116: /AUX21 -> /AUX23
- U16 pad 117: /AUX20 -> /AUX22
- U16 pad 118: /AUX19 -> /AUX21
- U16 pad 119: /AUX18 -> /AUX20
- U16 pad 120: /AUX17 -> /AUX19
- U16 pad 121: /AUX16 -> /AUX18
- U16 pad 122: /AUX15 -> /AUX17
- U16 pad 123: /AUX14 -> /AUX16
- U16 pad 127: /AUX13 -> /AUX15
- U16 pad 128: /AUX12 -> /AUX14
- U16 pad 13: /CAM2F -> /CAM1S
- U16 pad 131: /AUX11 -> /AUX13
- U16 pad 132: /AUX10 -> /AUX12
- U16 pad 133: /AUX09 -> /AUX11
- U16 pad 134: /AUX08 -> /AUX10
- U16 pad 135: /AUX07 -> /AUX09
- U16 pad 136: /AUX06 -> /AUX08
- U16 pad 137: /AUX05 -> /AUX07
- U16 pad 138: /AUX04 -> /AUX06
- U16 pad 139: (no net) -> /AUX05
- U16 pad 14: /CAM2S -> /CAM2F
- U16 pad 140: /AUX03 -> /AUX04
- U16 pad 141: /AUX02 -> /AUX03
- U16 pad 142: /CAM0F -> /AUX02
- U16 pad 143: /CAM0S -> /CAM0F
- U16 pad 144: /CAM1F -> /CAM0S
- U16 pad 15: /CAM3F -> /CAM2S
- U16 pad 16: /CAM3S -> /CAM3F
- U16 pad 19: /CAM4F -> /CAM3S
- U16 pad 20: /CAM4S -> /CAM4F
- U16 pad 21: /CAM5F -> /CAM4S
- U16 pad 22: /CAM5S -> /CAM5F
- U16 pad 23: /CAM6F -> /CAM5S
- U16 pad 24: /CAM6S -> /CAM6F
- U16 pad 25: /CAM7F -> /CAM6S
- U16 pad 26: /CAM7S -> /CAM7F
- U16 pad 32: (no net) -> /CAM7S
- U16 pad 55: /CC_RESET -> /CC_EXT1
- U16 pad 59: /CC_PROG -> /CC_EXT0
- U16 pad 60: /MOD3_ID -> /CC_RESET
- U16 pad 63: /MOD2_ID -> /CC_PROG
- U16 pad 64: /MOD1_ID -> /MOD3_ID
- U16 pad 65: /MOD0_ID -> /MOD2_ID
- U16 pad 66: /AUX47 -> /MOD1_ID
- U16 pad 67: /AUX46 -> /MOD0_ID
- U16 pad 68: /AUX45 -> /AUX47
- U16 pad 71: /AUX44 -> /AUX46
- U16 pad 72: /AUX43 -> /AUX45
- U16 pad 76: /AUX42 -> /AUX44
- U16 pad 77: /AUX41 -> /AUX43
- U16 pad 89: /AUX40 -> /AUX42
- U16 pad 90: /AUX39 -> /AUX41
- U16 pad 91: /AUX38 -> /AUX40
- U16 pad 92: /AUX37 -> /AUX39
- U16 pad 93: /AUX36 -> /AUX38
- U16 pad 94: /AUX35 -> /AUX37
- U16 pad 95: /AUX34 -> /AUX36
- U16 pad 96: /AUX33 -> /AUX35
- U16 pad 97: /AUX32 -> /AUX34
- U16 pad 98: /AUX31 -> /AUX33
- U16 pad 99: /AUX30 -> /AUX32
Routing:
- net GND: track 202.4 -> 209.4 mm, vias 74 -> 73
Other:
- board text added: "3V3"
- board text added: "Camera Axe 6 Version 4 March 26, 2017"
- board text added: "EXT0"
- board text added: "EXT1"
- board text added: "Reset"
- board text removed: "3.3V"
- board text removed: "Camera Axe 6 Version 4 March 10, 2017"
- board text removed: "RESET"
