File: Pcb/Cards/nRF52card.sch (KiCad schematic (older format))
At the start: 8 parts, among them J1 CA6_02X06, J2 NFC_ANT, J3 PROG_01X06, U1 SN74AHC1G08, U2 BL652-SA-01, X1 HOLE

Commit message: Updated all text on both ESP8266card and nRF52card to minimum of .635x.635x.1524 (6 mils).  Verified that all pins chosen on nRF52 can be used as general IO if we're not using smartBasic (which we probably won't be using), so I didn't change any of them.
Changed lines of the file:
@@
 Text Label 1600 4400 0    60   ~ 0
 CC_PROG
-Text Label 1600 5150 0    60   ~ 0
-nAUTORUN-not_sure-needed
 Wire Wire Line
 	8250 3500 8250 5100

Commit message: corrected labelling of EXT pins on both nRF52card and ESP8266card and rerouted some traces on nRF52card for better ground pour.
Parts:
- J1: footprint Pin_Headers:Pin_Header_Straight_2x06_Pitch2.54mm -> CA6:Pin_Header_Straight_2x06_Pitch2.54mm
- J3: footprint Pin_Headers:Pin_Header_Angled_1x06_Pitch2.54mm -> CA6:Pin_Header_Angled_1x06_Pitch2.54mm
- U1: footprint TO_SOT_Packages_SMD:SOT-23-5 -> CA6:SOT-23-5_GATE
Connections:
- net CC_EXT0: now also J1.11 (P11), U2.13 (SIO_11); no longer J1.12 (P12), U2.23 (SIO_02/AIN0)
- net CC_EXT1: now also J1.12 (P12), U2.23 (SIO_02/AIN0); no longer J1.11 (P11), U2.13 (SIO_11)
Changed lines of the file:
@@
 F 0 "J1" H 2300 4800 50  0000 C CNN
 F 1 "CA6_02X06" H 2300 4100 50  0000 C CNN
-F 2 "Pin_Headers:Pin_Header_Straight_2x06_Pitch2.54mm" H 2300 3250 50  0001 C CNN
+F 2 "CA6:Pin_Header_Straight_2x06_Pitch2.54mm" H 2300 3250 50  0001 C CNN
 F 3 "" H 2300 3250 50  0001 C CNN
 	1    2300 4450
@@
 Wire Wire Line
 	1700 4700 2050 4700
-Text Label 1750 4700 0    60   ~ 0
+Text Label 1700 4700 0    60   ~ 0
+CC_EXT0
+Text Label 2550 4700 0    60   ~ 0
 CC_EXT1
-Text Label 2550 4700 0    60   ~ 0
-CC_EXT0
 $Comp
 L PWR_FLAG #FLG08
@@
 F 0 "U1" H 4400 2150 50  0000 C CNN
 F 1 "SN74AHC1G08" H 4400 2050 50  0000 C CNN
-F 2 "TO_SOT_Packages_SMD:SOT-23-5" H 4350 1850 50  0001 C CNN
+F 2 "CA6:SOT-23-5_GATE" H 4350 1850 50  0001 C CNN
 F 3 "http://www.ti.com/lit/gpn/sn74ahc1g08" H 4400 2500 50  0001 C CNN
 	1    4400 2100
@@
 F 0 "J3" H 9050 5200 50  0000 C CNN
 F 1 "PROG_01X06" V 9150 4850 50  0000 C CNN
-F 2 "Pin_Headers:Pin_Header_Angled_1x06_Pitch2.54mm" H 9050 4850 50  0001 C CNN
+F 2 "CA6:Pin_Header_Angled_1x06_Pitch2.54mm" H 9050 4850 50  0001 C CNN
 F 3 "" H 9050 4850 50  0001 C CNN
 	1    9050 4850
