File: Pcb/Modules/Dev.kicad_pcb (KiCad board)
At the start: 2 copper layers, 38.1 x 38.1 mm, 9 parts, among them J1 JACK_STEREO, J2 JACK_RJ45, P1 CONN_02X04, P2 CONN_02X04, Q1 BSS138P, U1 11AA160, X1 HOLE, X2 HOLE

Commit message: Add new footprints for rj45 and switch
Parts:
- J2: footprint CA6:RJ45_RJHSE-5080 -> CA6:RJ45_pcbwing
Routing:
- net GND: track 14.3 -> 9.72 mm
Other:
- board text added: "Dev Module 2017-04-11"
- board text removed: "Dev Module 2017-04-03"
