File: Pcb/Modules/Dev.sch (KiCad schematic (older format))
At the start: 9 parts, among them J1 JACK_STEREO, J2 JACK_RJ45, P1 CONN_02X04, P2 CONN_02X04, Q1 BSS138P, U1 11AA160, X1 HOLE, X2 HOLE

Commit message: Add new footprints for rj45 and switch
Parts:
- J2: footprint CA6:RJ45_RJHSE-5080 -> CA6:RJ45_pcbwing
Changed lines of the file:
@@
 LIBS:valves
 LIBS:CA6
-LIBS:Dev-cache
 EELAYER 25 0
 EELAYER END
@@
 F 0 "J2" H 1325 2100 39  0000 C CNN
 F 1 "JACK_RJ45" H 975 2100 39  0000 C CNN
-F 2 "CA6:RJ45_RJHSE-5080" H 1125 1600 60  0001 C CNN
+F 2 "CA6:RJ45_pcbwing" H 1125 1600 60  0001 C CNN
 F 3 "" H 1125 1600 60  0000 C CNN
 	1    1150 1600
