File: Pcb/Modules/BeamEmit/BeamEmit.kicad_pcb (KiCad board)
At the start: 2 copper layers, 50.8 x 20.3 mm, 14 parts, among them J1 JACK_RJ45, Q1 Q_NMOS_GSD, X1 HOLE, X2 HOLE, X3 HOLE, X4 HOLE

Commit message: Update pcbs
Parts:
- moved R1 7.35 mm to (72.6, 43.4)
Routing:
- net +3V3: track 42.8 -> 36.3 mm
Changed lines of the file:
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@@
     (thickness 1.6)
     (drawings 14)
-    (tracks 61)
+    (tracks 60)
     (zones 0)
     (modules 14)
@@
   )
   (setup
-    (last_trace_width 0.254)
+    (last_trace_width 1.016)
     (user_trace_width 0.381)
     (user_trace_width 0.508)
@@
   )
   (module Resistors_SMD:R_1206 (layer F.Cu)
-    (at 79.629 45.72 180)
+    (at 72.644 43.434 180)
     (descr "Resistor SMD 1206, reflow soldering, Vishay (see dcrcw.pdf)")
     (tags "resistor 1206")
     (attr smd)
-    (fp_text reference R1 (at 0 2.032 180) (layer F.SilkS)
+    (fp_text reference R1 (at 3.302 0 180) (layer F.SilkS)
       (effects (font (size 1 1) (thickness 0.15)))
     )
@@
   (segment (start 79.248 48.26) (end 79.502 48.006) (width 1.016) (layer F.Cu) (net 4))
   (segment (start 79.502 42.164) (end 79.248 41.91) (width 1.016) (layer F.Cu) (net 4) (status 30))
-  (segment (start 79.248 39.37) (end 80.772 39.37) (width 1.016) (layer F.Cu) (net 5) (status 10))
-  (segment (start 81.788 45.011) (end 81.079 45.72) (width 1.016) (layer F.Cu) (net 5) (status 20))
-  (segment (start 81.788 40.386) (end 81.788 45.011) (width 1.016) (layer F.Cu) (net 5))
-  (segment (start 80.772 39.37) (end 81.788 40.386) (width 1.016) (layer F.Cu) (net 5))
-  (segment (start 78.179 45.72) (end 77.724 45.72) (width 1.016) (layer F.Cu) (net 6))
-  (segment (start 62.0192 48.4708) (end 58.42 48.4708) (width 1.016) (layer F.Cu) (net 6))
-  (segment (start 65.278 45.212) (end 62.0192 48.4708) (width 1.016) (layer F.Cu) (net 6))
-  (segment (start 77.216 45.212) (end 65.278 45.212) (width 1.016) (layer F.Cu) (net 6))
-  (segment (start 77.724 45.72) (end 77.216 45.212) (width 1.016) (layer F.Cu) (net 6))
+  (segment (start 74.094 43.434) (end 75.311 43.434) (width 1.016) (layer F.Cu) (net 5))
+  (segment (start 76.581 39.37) (end 79.248 39.37) (width 1.016) (layer F.Cu) (net 5))
+  (segment (start 76.2 39.751) (end 76.581 39.37) (width 1.016) (layer F.Cu) (net 5))
+  (segment (start 76.2 42.545) (end 76.2 39.751) (width 1.016) (layer F.Cu) (net 5))
+  (segment (start 75.311 43.434) (end 76.2 42.545) (width 1.016) (layer F.Cu) (net 5))
+  (segment (start 58.42 48.4708) (end 61.1302 48.4708) (width 1.016) (layer F.Cu) (net 6))
+  (segment (start 66.167 43.434) (end 71.194 43.434) (width 1.016) (layer F.Cu) (net 6))
+  (segment (start 61.1302 48.4708) (end 66.167 43.434) (width 1.016) (layer F.Cu) (net 6))
   (segment (start 58.42 48.4708) (end 58.8442 48.4708) (width 1.016) (layer F.Cu) (net 6))
   (segment (start 58.42 48.4708) (end 56.7258 48.4708) (width 1.016) (layer F.Cu) (net 6))
