File: Pcb/Modules/Valve/Valve.kicad_pcb (KiCad board)
At the start: 2 copper layers, 61 x 45.7 mm, 32 parts, among them J1 JACK_RJ45, Q1 Q_NMOS_GSD, Q2 Q_NMOS_GSD, Q3 Q_NMOS_GSD, Q4 Q_NMOS_GSD, X1 HOLE, X2 HOLE, X3 HOLE, X4 HOLE

Commit message: Update module pcbs to fix minor issues and round corners
Other:
- board text added: "1"
- board text added: "4"
- board text added: "Valve Module 2018.7.1"
- board text removed: "Valve Module 2018.3.31"
Changed lines of the file:
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@@
     (area 24.730999 23.411 86.849001 73.209)
     (thickness 1.6)
-    (drawings 9)
+    (drawings 11)
     (tracks 186)
     (zones 0)
@@
     (descr "DC Barrel Jack")
     (tags "Power Jack")
-    (fp_text reference Valve1 (at -10.922 5.334 450) (layer F.SilkS)
-      (effects (font (size 1 1) (thickness 0.15)))
+    (fp_text reference Valve1 (at -9.906 5.588 270) (layer F.SilkS)
+      (effects (font (thickness 0.254)))
     )
     (fp_text value Valve1 (at -6.2 -5.5 270) (layer F.Fab) hide
@@
     (descr "DC Barrel Jack")
     (tags "Power Jack")
-    (fp_text reference Valve2 (at -10.922 5.334 450) (layer F.SilkS)
-      (effects (font (size 1 1) (thickness 0.15)))
+    (fp_text reference Valve2 (at -9.906 5.588 270) (layer F.SilkS)
+      (effects (font (thickness 0.254)))
     )
     (fp_text value Valve2 (at -6.2 -5.5 270) (layer F.Fab) hide
@@
     (descr "DC Barrel Jack")
     (tags "Power Jack")
-    (fp_text reference Valve3 (at -10.922 5.334 450) (layer F.SilkS)
-      (effects (font (size 1 1) (thickness 0.15)))
+    (fp_text reference Valve3 (at -9.906 5.588 270) (layer F.SilkS)
+      (effects (font (thickness 0.254)))
     )
     (fp_text value Valve3 (at -6.2 -5.5 270) (layer F.Fab) hide
@@
     (descr "DC Barrel Jack")
     (tags "Power Jack")
-    (fp_text reference Valve4 (at -10.922 5.334 450) (layer F.SilkS)
-      (effects (font (size 1 1) (thickness 0.15)))
+    (fp_text reference Valve4 (at -9.906 5.588 270) (layer F.SilkS)
+      (effects (font (thickness 0.254)))
     )
     (fp_text value Valve4 (at -6.2 -5.5 270) (layer F.Fab) hide
@@
     (pad 1 thru_hole circle (at 0 0) (size 5 5) (drill 2.5) (layers *.Cu *.Mask))
   )
+  (gr_text 4 (at 83.82 35.56) (layer F.SilkS)
+    (effects (font (size 5.08 5.08) (thickness 1.016)))
+  )
+  (gr_text 1 (at 28.194 35.56) (layer F.SilkS)
+    (effects (font (size 5.08 5.08) (thickness 1.016)))
+  )
   (gr_line (start 26.67 25.4) (end 85.09 25.4) (angle 90) (layer Edge.Cuts) (width 0.15))
   (gr_line (start 85.09 71.12) (end 26.67 71.12) (angle 90) (layer Edge.Cuts) (width 0.15))
@@
   (gr_arc (start 26.67 26.67) (end 25.4 26.67) (angle 90) (layer Edge.Cuts) (width 0.15))
   (gr_arc (start 26.67 69.85) (end 26.67 71.12) (angle 90) (layer Edge.Cuts) (width 0.15))
-  (gr_text "Valve Module\n2018.3.31" (at 82.804 57.404 90) (layer F.SilkS)
+  (gr_text "Valve Module\n2018.7.1" (at 82.804 57.404 90) (layer F.SilkS)
     (effects (font (size 1.5 1.5) (thickness 0.3)))
   )
