File: Pcb/Modules/BeamDetect/BeamDetect.sch (KiCad schematic (older format))
At the start: 9 parts, among them J1 JACK_RJ45, U3 TSOP585xx, X1 HOLE, X2 HOLE, X3 HOLE, X4 HOLE

Commit message: Update pcb for new switch
Parts:
- C1: symbol CAP_ELEC -> CA6:CAP_ELEC
- C2: symbol C_Small -> Device:C_Small
- J1: symbol JACK_RJ45 -> CA6:JACK_RJ45
- R1: symbol R -> Device:R
- U3: symbol TSOP585xx -> opto:TSOP585xx
- X1, X2, X3, X4: symbol HOLE -> CA6:HOLE
Changed lines of the file:
@@
-EESchema Schematic File Version 2
-LIBS:power
-LIBS:device
-LIBS:switches
-LIBS:relays
-LIBS:motors
-LIBS:transistors
-LIBS:conn
-LIBS:linear
-LIBS:regul
-LIBS:74xx
-LIBS:cmos4000
-LIBS:adc-dac
-LIBS:memory
-LIBS:xilinx
-LIBS:microcontrollers
-LIBS:dsp
-LIBS:microchip
-LIBS:analog_switches
-LIBS:motorola
-LIBS:texas
-LIBS:intel
-LIBS:audio
-LIBS:interface
-LIBS:digital-audio
-LIBS:philips
-LIBS:display
-LIBS:cypress
-LIBS:siliconi
-LIBS:opto
-LIBS:atmel
-LIBS:contrib
-LIBS:valves
-LIBS:CA6
-LIBS:Beam-cache
-EELAYER 25 0
+EESchema Schematic File Version 4
+LIBS:BeamDetect-cache
+EELAYER 26 0
 EELAYER END
 $Descr A4 11693 8268
@@
 $EndDescr
 $Comp
-L TSOP585xx U3
+L opto:TSOP585xx U3
 U 1 1 59CD457D
 P 6850 1650
@@
 $EndComp
 $Comp
-L +3.3V #PWR01
+L power:+3.3V #PWR01
 U 1 1 59FCE3A1
 P 4500 2050
@@
 $EndComp
 $Comp
-L GND #PWR02
+L power:GND #PWR02
 U 1 1 59FCE5A5
 P 4500 2850
@@
 $EndComp
 $Comp
-L C_Small C2
+L Device:C_Small C2
 U 1 1 59FD6427
 P 6100 1900
@@
 $EndComp
 $Comp
-L GND #PWR03
+L power:GND #PWR03
 U 1 1 59FD6B4A
 P 6100 2100
@@
 $EndComp
 $Comp
-L +3.3V #PWR04
+L power:+3.3V #PWR04
 U 1 1 59FD6C0D
 P 5150 1300
@@
 $EndComp
 Wire Wire Line
-	5450 1450 6450 1450
+	5450 1450 5650 1450
 Wire Wire Line
 	5150 1300 5150 1450
@@
 	6100 2000 6100 2100
 $Comp
-L GND #PWR05
+L power:GND #PWR05
 U 1 1 59FD6E29
 P 6450 2100
@@
 	4750 2200 4350 2200
 $Comp
-L JACK_RJ45 J1
+L CA6:JACK_RJ45 J1
 U 1 1 59FCD911
 P 3900 2450
@@
 NoConn ~ 4350 2700
 $Comp
-L R R1
+L Device:R R1
 U 1 1 5A21DC3C
 P 5300 1450
@@
 $EndComp
 $Comp
-L CAP_ELEC C1
+L CA6:CAP_ELEC C1
 U 1 1 5A21DD7D
 P 5650 2050
@@
 Connection ~ 5650 1450
 $Comp
-L GND #PWR06
+L power:GND #PWR06
 U 1 1 5A21DE51
 P 5650 2250
@@
 NoConn ~ 4350 2300
 $Comp
-L HOLE X1
+L CA6:HOLE X1
 U 1 1 5A22D009
 P 5750 3150
@@
 $EndComp
 $Comp
-L HOLE X2
+L CA6:HOLE X2
 U 1 1 5A22D141
 P 6050 3150
@@
 $EndComp
 $Comp
-L HOLE X3
+L CA6:HOLE X3
 U 1 1 5A22D16C
 P 6350 3150
@@
 $EndComp
 $Comp
-L HOLE X4
+L CA6:HOLE X4
 U 1 1 5A22D1A0
 P 6650 3150
@@
 	1    0    0    -1
 $EndComp
+Wire Wire Line
+	6100 1450 6450 1450
+Wire Wire Line
+	5650 1450 6100 1450
 $EndSCHEMATC
